File: RS485iso.kicad_sch (KiCad schematic)
At the start: 12 parts, among them U11 ISO3082DW

Commit message: asdf
Parts:
- added C31, C32, C33, C34: C_Small, symbol Device:C_Small
- added U10: ADuM5411, Package_SO:SSOP-24_5.3x8.2mm_P0.65mm, symbol Isolator:ADuM5411
- added U12: ISO7331C, Package_SO:SOIC-16W_7.5x10.3mm_P1.27mm, symbol Isolator:ISO7331C
- added U9: ADuM6000, symbol Regulator_Switching:ADuM6000
Connections:
- net GND: now also C31.2, C32.2, U9.2 (GND1), U9.8 (GND1)
- net Vin: now also C31.1, C32.1, U9.1 (VDD1), U9.7 (VDD1)
- net ex5V: now also C33.1, C34.1, U9.10 (V_ISO), U9.16 (V_ISO)
- net exGND: now also C33.2, C34.2, U9.15 (GND_ISO), U9.9 (GND_ISO)
- new net: U10.12 (GND1), U10.2 (GND1), U10.9 (GND1)
- new net: U10.13 (GNDISO), U10.16 (GNDISO), U10.23 (GNDISO)
Other:
- note added: "ADUM8572 RS485 Isolated Receiver with isolatet power"
