File: hw_voltmod.kicad_pcb (KiCad board)
At the start: 2 copper layers, 70 x 50 mm, 96 parts, among them J1 Conn_01x09_Pin, J2 Conn_01x05_Pin, J3 Conn_01x04_Pin, U1 L78L33_SO8, U2 STM32G071KBTx, U3 TL074, U4 TL074

Commit message: 654
Parts:
- added D6: BAT41, Diode_SMD:D_0805_2012Metric_Pad1.15x1.40mm_HandSolder, B.Cu at (5.00, 17.5)
- added D7: BAT41, Diode_SMD:D_0805_2012Metric_Pad1.15x1.40mm_HandSolder, B.Cu at (5.00, 22.5)
- added D8: BAT41, Diode_SMD:D_0805_2012Metric_Pad1.15x1.40mm_HandSolder, B.Cu at (5.00, 27.5)
- added D9: BAT41, Diode_SMD:D_0805_2012Metric_Pad1.15x1.40mm_HandSolder, B.Cu at (5.00, 12.5)
- C1: footprint Capacitor_SMD:CP_Elec_5x3 -> Capacitor_SMD:C_1206_3216Metric_Pad1.33x1.80mm_HandSolder
- D1, D2, D3, D4, D5: footprint Diode_SMD:D_SOD-323_HandSoldering -> Diode_SMD:D_0805_2012Metric_Pad1.15x1.40mm_HandSolder; moved to B.Cu
- moved JP1 65.4 mm to (3.25, 2.98), turned to 90 degrees
- moved U1 63.1 mm to (17.0, 4.13), turned to 180 degrees
- moved C1 47.4 mm to (11.5, 4.50), turned to 90 degrees
- moved D5 31.9 mm to (5.00, 15.0)
- moved D1 26.7 mm to (5.03, 10.0)
- moved D4 25.8 mm to (5.00, 20.0)
- moved C2 20.2 mm to (9.00, 3.50), turned to 90 degrees
- moved D2 18.6 mm to (5.00, 30.0)
- moved D3 18.4 mm to (5.00, 25.0)
Routing:
- net Net-(D1-K): track 0.00 -> 27.3 mm
- net GNDD: track 0.00 -> 21.9 mm
- net VBUS: track 0.00 -> 10.8 mm
- net /Level Shifter/cell7: track 7.88 -> 2.94 mm
- net /Level Shifter/cell8: track 4.93 -> 0.00 mm

Commit message: asdf
Parts:
- removed C14, C18, C24, C6: 100n, Capacitor_SMD:C_0603_1608Metric_Pad1.08x0.95mm_HandSolder
- removed R13, R6: 47k, Resistor_SMD:R_0603_1608Metric_Pad0.98x0.95mm_HandSolder
- moved R23 93.6 mm to (37.0, 34.0), turned to 180 degrees
- moved R7 92.0 mm to (30.5, 34.0)
- moved R31 89.9 mm to (37.0, 32.0)
- moved R14 88.8 mm to (30.5, 32.0)
- moved R45 86.2 mm to (37.0, 19.0)
- moved R36 85.9 mm to (37.0, 17.0), turned to 180 degrees
- moved R57 75.6 mm to (31.0, 19.0), turned to 180 degrees
- moved R54 75.1 mm to (31.0, 17.0)
- moved R5 3.35 mm to (23.5, 31.0)
- moved R12 1.80 mm to (23.5, 29.0)
- moved R30 1.59 mm to (23.4, 23.0)
- moved R22 1.58 mm to (23.5, 25.5)
- moved C16 0.50 mm to (20.0, 24.5)
- moved R11 0.50 mm to (16.0, 28.4)
- moved R21 0.50 mm to (16.0, 25.5)
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Connections:
- R14 pad 2: Net-(R13-Pad1) -> Net-(U3A--)
- R7 pad 2: Net-(R6-Pad1) -> Net-(U3A-+)
Routing:
- net Net-(C8-Pad2): track 10.5 -> 0.35 mm
- net Net-(U3A-+): track 9.17 -> 0.81 mm
- net Net-(C8-Pad1): track 8.03 -> 0.00 mm
- net Net-(U3A--): track 6.74 -> 1.00 mm
- net /Level Shifter/cell8_amp: track 4.96 -> 0.00 mm
- net /Level Shifter/cell7: track 2.94 -> 0.00 mm
